File: DgDrive_DVI.kicad_pcb (KiCad board)
At the start: 2 copper layers, 69 x 28 mm, 41 parts, among them J1 Curr. Mod., J2 DVI-I, J3 Ld+, J4 Ld-, J5 Pz+, J6 Pz-, J7 Piezo_In, K1 G6AU, Q1 MMBT3904, Q2 2N4401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

Commit message: SMD solder pads for piezo connection
Parts:
- J5, J6: footprint Connector_Wire:SolderWirePad_1x01_Drill1mm -> TestPoint:TestPoint_Keystone_5015_Micro-Minature
- R3: value 1k -> 100k
- moved J6 2.08 mm to (155.7, 93.1)
- turned J5 to 180 degrees
Other:
- board text added: "LaserBackplane Diode DVI 11/2021 Rev 1.6"
- board text added: "Rev. 1.6"
- board text removed: "LaserBackplane Diode DVI 10/2021 Rev 1.6"

Commit message: Update PCB
Parts:
- added C5: DNF, Capacitor_SMD:C_0603_1608Metric, F.Cu at (140.3, 116.1)
- added C6: 10n, Capacitor_SMD:C_0603_1608Metric, F.Cu at (121.4, 104.0)
- added R6: 1k, Resistor_SMD:R_0603_1608Metric, F.Cu at (143.8, 116.9)
- added R9: 4.7, Resistor_SMD:R_0603_1608Metric, F.Cu at (124.6, 104.0)
Connections:
- net Net-(J2-Pad10) renamed Ld+
- U1 pad 3: Net-(J1-Pad1) -> Net-(C5-Pad2)
Routing:
- net Net-(J1-Pad1): track 19.3 -> 9.55 mm
- net Net-(C5-Pad2): track 0.00 -> 7.66 mm
- net GND: track 23.9 -> 31.2 mm
- net Net-(C6-Pad1): track 0.00 -> 1.62 mm
- net LD_short-: track 50.8 -> 50.2 mm
Other:
- board text added: "LaserBackplane Diode DVI 12/2021 Rev 1.7"
- board text added: "Rev. 1.7"
- board text removed: "LaserBackplane Diode DVI 11/2021 Rev 1.6"
- board text removed: "Rev. 1.6"
