File: DgDrive_DVI.kicad_pcb (KiCad board)
At the start: 2 copper layers, 69 x 28 mm, 45 parts, among them J1 Curr. Mod., J2 DVI-I, J3 Ld+, J4 Ld-, J5 Pz+, J6 Pz-, J7 Piezo_In, K1 G6AU, Q1 MMBT3904, Q2 2N4401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

Commit message: Update to KiCad6
Parts:
- moved R9 0.17 mm to (124.8, 104.0)
Connections:
- J2 pad 1: Net-(J2-Pad1) -> unconnected-(J2-Pad1)
- J2 pad 11: Net-(J2-Pad11) -> unconnected-(J2-Pad11)
- J2 pad 17: Net-(J2-Pad17) -> unconnected-(J2-Pad17)
- J2 pad 18: Net-(J2-Pad18) -> unconnected-(J2-Pad18)
- J2 pad 19: Net-(J2-Pad19) -> unconnected-(J2-Pad19)
- J2 pad 2: Net-(J2-Pad2) -> unconnected-(J2-Pad2)
- J2 pad 20: Net-(J2-Pad20) -> unconnected-(J2-Pad20)
- J2 pad 21: Net-(J2-Pad21) -> unconnected-(J2-Pad21)
- J2 pad 22: Net-(J2-Pad22) -> unconnected-(J2-Pad22)
- J2 pad 3: Net-(J2-Pad3) -> unconnected-(J2-Pad3)
- J2 pad 4: Net-(J2-Pad4) -> unconnected-(J2-Pad4)
- J2 pad 5: Net-(J2-Pad5) -> unconnected-(J2-Pad5)
- J2 pad 8: Net-(J2-Pad8) -> unconnected-(J2-Pad8)
- J2 pad C1: Net-(J2-PadC1) -> unconnected-(J2-PadC1)
- J2 pad C2: Net-(J2-PadC2) -> unconnected-(J2-PadC2)
- J2 pad C3: Net-(J2-PadC3) -> unconnected-(J2-PadC3)
- J2 pad C4: Net-(J2-PadC4) -> unconnected-(J2-PadC4)
- J2 pad C5: Net-(J2-PadC5) -> unconnected-(J2-PadC5)
- J2 pad SH: Net-(J2-PadSH) -> unconnected-(J2-PadSH)
- K1 pad 11: Net-(K1-Pad11) -> unconnected-(K1-Pad11)
- K1 pad 8: Net-(K1-Pad8) -> unconnected-(K1-Pad8)
- U4 pad 2: Net-(U4-Pad2) -> unconnected-(U4-Pad2)
Routing:
- net Curr_Mod: track 40.7 -> 39.9 mm
- net LD_short-: track 50.2 -> 49.5 mm
- net Net-(R4-Pad1): track 12.0 -> 11.5 mm
Other:
- net class Default removed
- board text added: "LaserBackplane Diode DVI 01/2022 Rev 1.7"
- board text removed: "LaserBackplane Diode DVI 12/2021 Rev 1.7"
