File: DgDrive_DVI.kicad_sch (KiCad schematic)
At the start: 45 parts, among them J1 Curr. Mod., J2 DVI-I, J3 Ld+, J4 Ld-, J5 Pz+, J6 Pz-, J7 Piezo_In, K1 G6AU, Q1 MMBT3904, Q2 2N4401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

Commit message: Update DVI connector 3D model
Parts:
- U1: MFN (none) -> Analog Devices; PN (none) -> ADA4807-2ARMZ
- U2, U3: MFN Linear Technology -> Analog Devices
Changed lines of the file:
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@@
     (pin "2")
   )
-  (symbol (lib_id "Device:R") (at 165.1 52.07 180)
+  (symbol (lib_id "Device:R") (at 165.1 52.07 180) (unit 1)
     (in_bom yes) (on_board yes)
     (property "Reference" "R5" (id 0) (at 162.56 53.34 0)
@@
     (pin "2")
   )
-  (symbol (lib_id "Device:D") (at 73.66 24.13 180)
+  (symbol (lib_id "Device:D") (at 73.66 24.13 180) (unit 1)
     (in_bom yes) (on_board yes)
     (property "Reference" "D1" (id 0) (at 73.66 17.78 0))
@@
     )
   )
-  (symbol (lib_id "Device:R") (at 198.12 77.47 180)
+  (symbol (lib_id "Device:R") (at 198.12 77.47 180) (unit 1)
     (in_bom yes) (on_board yes)
     (property "Reference" "R7" (id 0) (at 195.58 78.74 0)
@@
     (pin "2")
   )
-  (symbol (lib_id "Device:R") (at 198.12 102.87 180)
+  (symbol (lib_id "Device:R") (at 198.12 102.87 180) (unit 1)
     (in_bom yes) (on_board yes)
     (property "Reference" "R8" (id 0) (at 195.58 104.14 0)
@@
       (effects (font (size 1.27 1.27)) hide)
     )
-    (property "MFN" "Linear Technology" (id 4) (at 171.45 143.51 0)
+    (property "MFN" "Analog Devices" (id 4) (at 171.45 143.51 0)
       (effects (font (size 1.27 1.27)) hide)
     )
@@
       (effects (font (size 1.27 1.27)) hide)
     )
-    (property "MFN" "Linear Technology" (id 4) (at 242.57 143.51 0)
+    (property "MFN" "Analog Devices" (id 4) (at 242.57 143.51 0)
       (effects (font (size 1.27 1.27)) hide)
     )
@@
       (effects (font (size 1.27 1.27)) hide)
     )
+    (property "MFN" "Analog Devices" (id 4) (at 147.32 176.53 0)
+      (effects (font (size 1.27 1.27)) hide)
+    )
+    (property "PN" "ADA4807-2ARMZ" (id 5) (at 147.32 176.53 0)
+      (effects (font (size 1.27 1.27)) hide)
+    )
     (pin "4")
     (pin "8")
@@
     (pin "1")
   )
-  (symbol (lib_id "Device:R_Small") (at 43.18 161.29 90)
+  (symbol (lib_id "Device:R_Small") (at 43.18 161.29 90) (unit 1)
     (in_bom yes) (on_board yes)
     (property "Reference" "R6" (id 0) (at 41.91 158.75 0)
